Commit message: World

File: models/urdf/lidar.urdf.xacro (robot description, xacro)
@@ -12,5 +12,5 @@
       <origin xyz="0 0 1.0" rpy="0 0 0"/>
       <geometry>
-        <mesh filename="$(find lidar_samples)/models/meshes/sensors/lds.stl" scale="0.001 0.001 0.001"/>
+        <mesh filename="package://lidar_samples/models/meshes/lds.stl" scale="0.001 0.001 0.001"/>
       </geometry>
       <material name="dark"/>
